File: Hardware/Schaltplan/KiCad_Wecker_2v0/Wecker_2v0.kicad_sch (KiCad schematic)
At the start: 48 parts, among them J1 USB_C_Receptacle_PowerOnly_6P, J2 Conn_01x02_Pin, J3 Conn_01x02_Pin, J4 Conn_01x02_Pin, M1 Mühlrad, Q1 IRLML6344, Q2 IRLML6344, Q3 IRLML6344, U1 SSD1306-I2C, U2 DFPlayer_MiniMP3, U3 ESP32DevKitCv4, U4 MCP1700T-1502E/MB, U5 MCP1700T-3302E/TO

Commit message: Firmware 20v28: Taster S1/S2 GPIO getauscht (Schaltplan-Update Hardware 2v0)
S1 (Alarm aus / Kuckuck einmalig) liegt jetzt auf GPIO33, S2 (Zugschalter
Licht + Muehlrad) auf GPIO32. Nur die Pin-Zuordnung in SysConf_20v28.h
(S1/S2/EVT_S1/EVT_S2) angepasst - Event-/State-Logik (isrS1()/isrS2(),
inputTask) arbeitet ausschliesslich mit den symbolischen Konstanten und
bleibt unveraendert.
Parts:
- LS1: value Speaker -> FRWS 4 ND
Other:
- note added: "Treppentaster"
- note added: "VISATON"
- note added: "Zugschalter"
- note added: "ge"
- note added: "gn"
- moved on the sheet: LS1
Changed lines of the file:
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@@
+		)
+	)
+	(text "ge"
+		(exclude_from_sim no)
+		(at 46.736 87.63 0)
+		(effects
+			(font
+				(size 1.27 1.27)
+			)
 		)
 	)
@@
 	(text "Player Modul"
 		(exclude_from_sim no)
-		(at 91.44 23.622 0)
+		(at 52.07 19.304 0)
 		(effects
 			(font
@@
 		)
 	)
+	(text "Treppentaster"
+		(exclude_from_sim no)
+		(at 178.054 103.886 0)
+		(effects
+			(font
+				(size 1 1)
+			)
+		)
+	)
+	(text "VISATON"
+		(exclude_from_sim no)
+		(at 41.402 90.678 0)
+		(effects
+			(font
+				(size 1.27 1.27)
+			)
+		)
+	)
 	(text "Touch Modul"
 		(exclude_from_sim no)
@@
 		)
 	)
-	(text_box ""
+	(text "gn"
 		(exclude_from_sim no)
-		(at 80.01 181.61 0)
-		(size 49.53 12.7)
-		(margins 1.75 1.75 1.75 1.75)
-		(stroke
-			(width 0.5)
-			(type default)
-		)
-		(fill
-			(type color)
-			(color 255 246 180 1)
-		)
+		(at 46.736 82.55 0)
 		(effects
 			(font
-				(face "KiCad Font")
-				(size 2 2)
+				(size 1.27 1.27)
+			)
+		)
+	)
+	(text "Zugschalter"
+		(exclude_from_sim no)
+		(at 161.29 103.632 0)
+		(effects
+			(font
+				(size 1 1)
 			)
 		)
@@
 		)
 	)
-	(text_box ""
-		(exclude_from_sim no)
-		(at 50.8 20.32 0)
-		(size 52.07 72.39)
-		(margins 1.75 1.75 1.75 1.75)
-		(stroke
-			(width 0.5)
-			(type default)
-		)
-		(fill
-			(type color)
-			(color 255 246 180 1)
-		)
-		(effects
-			(font
-				(face "KiCad Font")
-				(size 2 2)
-			)
-		)
-	)
 	(text_box "Cuckoo Modul"
 		(exclude_from_sim no)
@@
 	(wire
 		(pts
-			(xy 53.34 86.36) (xy 48.26 86.36)
+			(xy 53.34 86.36) (xy 44.45 86.36)
 		)
 		(stroke
@@
 	(wire
 		(pts
-			(xy 86.36 53.34) (xy 86.36 69.85)
+			(xy 86.36 54.61) (xy 86.36 69.85)
 		)
 		(stroke
@@
 	(wire
 		(pts
-			(xy 53.34 83.82) (xy 48.26 83.82)
+			(xy 53.34 83.82) (xy 44.45 83.82)
 		)
 		(stroke
@@
 	(wire
 		(pts
-			(xy 143.51 97.79) (xy 143.51 53.34)
-		)
-		(stroke
-			(width 0)
-			(type default)
-		)
-	)
-	(wire
-		(pts
-			(xy 143.51 53.34) (xy 86.36 53.34)
+			(xy 143.51 97.79) (xy 143.51 54.61)
+		)
+		(stroke
+			(width 0)
+			(type default)
+		)
+	)
+	(wire
+		(pts
+			(xy 143.51 54.61) (xy 86.36 54.61)
 		)
 		(stroke
@@
 		(polyline
 			(pts
-				(xy 187.96 99.06) (xy 187.96 118.11) (xy 276.86 118.11) (xy 276.86 143.51) (xy 168.91 143.51) (xy 168.91 99.06)
+				(xy 50.8 16.51) (xy 233.68 16.51) (xy 233.68 52.07) (xy 102.87 52.07) (xy 102.87 92.71) (xy 50.8 92.71)
 			)
 			(stroke
@@
 			)
 			(fill
-				(type none)
+				(type color)
+				(color 180 255 143 0.1019607843)
+			)
+		)
+	)
+	(rule_area
+		(exclude_from_sim no)
+		(in_bom yes)
+		(on_board yes)
+		(dnp no)
+		(polyline
+			(pts
+				(xy 187.96 99.06) (xy 187.96 118.11) (xy 276.86 118.11) (xy 276.86 143.51) (xy 168.91 143.51) (xy 168.91 99.06)
+			)
+			(stroke
+				(width 0)
+				(type dash)
+			)
+			(fill
+				(type color)
+				(color 180 255 143 0.1019607843)
+			)
+		)
+	)
+	(rule_area
+		(exclude_from_sim no)
+		(in_bom yes)
+		(on_board yes)
+		(dnp no)
+		(polyline
+			(pts
+				(xy 80.01 181.61) (xy 129.54 181.61) (xy 129.54 194.31) (xy 80.01 194.31)
+			)
+			(stroke
+				(width 0)
+				(type dash)
+			)
+			(fill
+				(type color)
+				(color 85 255 0 0.1019607843)
 			)
 		)
@@
 	(symbol
 		(lib_id "Device:Speaker")
-		(at 43.18 86.36 180)
+		(at 39.37 86.36 180)
 		(unit 1)
 		(body_style 1)
@@
 		(dnp no)
 		(property "Reference" "LS1"
-			(at 43.434 75.692 0)
+			(at 39.624 75.692 0)
 			(show_name no)
 			(do_not_autoplace no)
@@
 			)
 		)
-		(property "Value" "Speaker"
-			(at 47.244 78.232 0)
+		(property "Value" "FRWS 4 ND"
+			(at 43.434 78.232 0)
 			(show_name no)
 			(do_not_autoplace no)
@@
 		)
 		(property "Footprint" ""
-			(at 43.18 81.28 0)
+			(at 39.37 81.28 0)
 			(hide yes)
 			(show_name no)
@@
 		)
 		(property "Datasheet" ""
-			(at 43.434 85.09 0)
+			(at 39.624 85.09 0)
 			(hide yes)
 			(show_name no)
@@
 		)
 		(property "Description" ""
-			(at 43.18 86.36 0)
+			(at 39.37 86.36 0)
 			(show_name no)
 			(do_not_autoplace no)
