File: Hardware/Schaltplan/KiCad_Wecker_2v0/Wecker_2v0.kicad_pcb (KiCad board)
At the start: 2 copper layers, 50 parts

Commit message: Hardware: KiCad-Layout 2v0 aktualisiert, Pin_GPIO-Liste mit PIN-Nummern, Fotos Lautsprecher-Modul, Layout.pdf
Co-Authored-By: Claude Sonnet 5.5 <noreply@anthropic.com>
Parts:
- removed the REF** at (74.9, 80.0)
- removed the REF** at (49.5, 54.6)
- removed the REF** at (29.2, 44.4)
- removed the REF** at (36.8, 64.8)
- removed the REF** at (31.8, 36.8)
- removed the REF** at (52.1, 64.8)
- removed the REF** at (67.3, 57.1)
- removed the REF** at (77.5, 57.1)
- removed the REF** at (62.2, 54.6)
- removed the REF** at (59.7, 54.6)
- removed the REF** at (77.5, 54.6)
- removed the REF** at (31.8, 41.9)
- removed the REF** at (67.3, 54.6)
- removed the REF** at (31.8, 57.1)
- removed the REF** at (85.1, 54.6)
- removed the REF** at (31.8, 39.4)
- removed the REF** at (62.2, 72.4)
- removed the REF** at (62.2, 57.1)
- removed the REF** at (80.0, 54.6)
- removed the REF** at (64.8, 57.1)
- removed the REF** at (34.3, 57.1)
- removed the REF** at (29.2, 57.1)
- removed the REF** at (41.5, 59.7)
- removed the REF** at (40.2, 53.3)
- removed the REF** at (41.5, 54.6)
- removed the REF** at (40.2, 63.5)
- removed the REF** at (41.5, 64.8)
- removed the REF** at (40.2, 58.4)
- removed the REF** at (34.3, 44.4)
- removed the REF** at (31.8, 44.4)
- removed the REF** at (74.9, 74.9)
- removed the REF** at (59.7, 57.1)
- added R15: 1k, Resistor_THT:R_Axial_DIN0207_L6.3mm_D2.5mm_P10.16mm_Horizontal, F.Cu at (80.0, 59.7)
- added REF**: R_Axial_DIN0207_L6.3mm_D2.5mm_P10.16mm_Horizontal, Resistor_THT:R_Axial_DIN0207_L6.3mm_D2.5mm_P10.16mm_Horizontal, F.Cu at (69.8, 57.1)
- added REF**: 10µF, Capacitor_THT:C_Disc_D3.0mm_W1.6mm_P2.50mm, F.Cu at (52.1, 64.8)
- added REF**: 1,5V, Connector_Pin:Pin_D1.0mm_L10.0mm, F.Cu at (59.7, 57.1)
- added REF**: R_Axial_DIN0207_L6.3mm_D2.5mm_P10.16mm_Horizontal, Resistor_THT:R_Axial_DIN0207_L6.3mm_D2.5mm_P10.16mm_Horizontal, F.Cu at (62.2, 57.1)
- added REF**: GPIO 13, Connector_Pin:Pin_D1.0mm_L10.0mm, F.Cu at (245.1, 64.8)
- added REF**: R_Axial_DIN0207_L6.3mm_D2.5mm_P10.16mm_Horizontal, Resistor_THT:R_Axial_DIN0207_L6.3mm_D2.5mm_P10.16mm_Horizontal, F.Cu at (242.6, 64.8)
- added REF**: R_Axial_DIN0207_L6.3mm_D2.5mm_P10.16mm_Horizontal, Resistor_THT:R_Axial_DIN0207_L6.3mm_D2.5mm_P10.16mm_Horizontal, F.Cu at (242.6, 62.2)
- added REF**: PinHeader_1x11_P2.54mm_Vertical, Connector_PinHeader_2.54mm:PinHeader_1x11_P2.54mm_Vertical, F.Cu at (181.6, 44.5)
- added REF**: R_Axial_DIN0207_L6.3mm_D2.5mm_P10.16mm_Horizontal, Resistor_THT:R_Axial_DIN0207_L6.3mm_D2.5mm_P10.16mm_Horizontal, F.Cu at (67.3, 57.1)
- added REF**: BUSY, Connector_Pin:Pin_D1.0mm_L10.0mm, F.Cu at (77.5, 57.1)
- added REF**: BUSY, Connector_Pin:Pin_D1.0mm_L10.0mm, F.Cu at (227.3, 44.5)
- added REF**: Display SDA, Connector_Pin:Pin_D1.0mm_L10.0mm, F.Cu at (257.8, 44.5)
- added REF**: LED, Connector_Pin:Pin_D1.0mm_L10.0mm, F.Cu at (41.9, 59.7)
- added REF**: GPIO 33, Connector_Pin:Pin_D1.0mm_L10.0mm, F.Cu at (227.3, 49.5)
- added REF**: RX, Connector_Pin:Pin_D1.0mm_L10.0mm, F.Cu at (64.8, 57.1)
- added REF**: GND, Connector_Pin:Pin_D1.0mm_L10.0mm, F.Cu at (52.1, 67.3)
- added REF**: C_Rect_L7.0mm_W2.0mm_P5.00mm, Capacitor_THT:C_Rect_L7.0mm_W2.0mm_P5.00mm, F.Cu at (52.1, 62.2)
- added REF**: gn SPK-, Connector_Pin:Pin_D1.0mm_L10.0mm, F.Cu at (74.9, 80.0)
- added REF**: GPIO 4, Connector_Pin:Pin_D1.0mm_L10.0mm, F.Cu at (240.0, 62.2)
- added REF**: 3V3, Connector_Pin:Pin_D1.0mm_L10.0mm, F.Cu at (229.9, 31.8)
- added REF**: R_Axial_DIN0207_L6.3mm_D2.5mm_P10.16mm_Horizontal, Resistor_THT:R_Axial_DIN0207_L6.3mm_D2.5mm_P10.16mm_Horizontal, F.Cu at (36.8, 57.1)
- added REF**: Motor, Connector_Pin:Pin_D1.0mm_L10.0mm, F.Cu at (41.9, 64.8)
- added REF**: RX, Connector_Pin:Pin_D1.0mm_L10.0mm, F.Cu at (257.8, 57.1)
- added REF**: R_Axial_DIN0207_L6.3mm_D2.5mm_P10.16mm_Horizontal, Resistor_THT:R_Axial_DIN0207_L6.3mm_D2.5mm_P10.16mm_Horizontal, F.Cu at (242.6, 69.8)
- added REF**: GND, Connector_Pin:Pin_D1.0mm_L10.0mm, F.Cu at (47.0, 74.9)
- added REF**: R_Axial_DIN0207_L6.3mm_D2.5mm_P10.16mm_Horizontal, Resistor_THT:R_Axial_DIN0207_L6.3mm_D2.5mm_P10.16mm_Horizontal, F.Cu at (34.3, 39.4)
- added REF**: R_Axial_DIN0207_L6.3mm_D2.5mm_P10.16mm_Horizontal, Resistor_THT:R_Axial_DIN0207_L6.3mm_D2.5mm_P10.16mm_Horizontal, F.Cu at (242.6, 67.3)
- added REF**: C_Rect_L7.0mm_W2.0mm_P5.00mm, Capacitor_THT:C_Rect_L7.0mm_W2.0mm_P5.00mm, F.Cu at (80.0, 57.1)
- added REF**: R_Axial_DIN0207_L6.3mm_D2.5mm_P10.16mm_Horizontal, Resistor_THT:R_Axial_DIN0207_L6.3mm_D2.5mm_P10.16mm_Horizontal, F.Cu at (34.3, 41.9)
- added REF**: GPIO 27, Connector_Pin:Pin_D1.0mm_L10.0mm, F.Cu at (39.4, 44.4)
- added REF**: GPIO 2, Connector_Pin:Pin_D1.0mm_L10.0mm, F.Cu at (240.0, 67.3)
- added REF**: GPIO 26, Connector_Pin:Pin_D1.0mm_L10.0mm, F.Cu at (36.8, 44.4)
- added REF**: GPIO 15, Connector_Pin:Pin_D1.0mm_L10.0mm, F.Cu at (240.0, 69.8)
- added REF**: TX, Connector_Pin:Pin_D1.0mm_L10.0mm, F.Cu at (257.8, 59.7)
- added REF**: RX, Connector_Pin:Pin_D1.0mm_L10.0mm, F.Cu at (257.8, 47.0)
- added REF**: Vcc, Connector_Pin:Pin_D1.0mm_L10.0mm, F.Cu at (229.9, 77.5)
- added REF**: R_Axial_DIN0207_L6.3mm_D2.5mm_P10.16mm_Horizontal, Resistor_THT:R_Axial_DIN0207_L6.3mm_D2.5mm_P10.16mm_Horizontal, F.Cu at (34.3, 36.8)
- added REF**: LED+, Connector_Pin:Pin_D1.0mm_L10.0mm, F.Cu at (59.7, 67.3)
- added REF**: GND, Connector_Pin:Pin_D1.0mm_L10.0mm, F.Cu at (54.6, 57.1)
- added REF**: R_Axial_DIN0207_L6.3mm_D2.5mm_P10.16mm_Horizontal, Resistor_THT:R_Axial_DIN0207_L6.3mm_D2.5mm_P10.16mm_Horizontal, F.Cu at (39.4, 57.1)
- added REF**: TX, Connector_Pin:Pin_D1.0mm_L10.0mm, F.Cu at (72.4, 57.1)
- added REF**: GPIO 25, Connector_Pin:Pin_D1.0mm_L10.0mm, F.Cu at (34.3, 44.4)
- added REF**: Vcc, Connector_Pin:Pin_D1.0mm_L10.0mm, F.Cu at (64.8, 62.2)
- added REF**: GPIO 32, Connector_Pin:Pin_D1.0mm_L10.0mm, F.Cu at (227.3, 47.0)
- added REF**: ge SPK+, Connector_Pin:Pin_D1.0mm_L10.0mm, F.Cu at (74.9, 74.9)
- added REF**: GPIO 25, Connector_Pin:Pin_D1.0mm_L10.0mm, F.Cu at (227.3, 52.1)
- added REF**: CP_Radial_D8.0mm_P5.00mm, Capacitor_THT:CP_Radial_D8.0mm_P5.00mm, F.Cu at (64.8, 69.9)
- added REF**: CUCKOO, Connector_Pin:Pin_D1.0mm_L10.0mm, F.Cu at (41.9, 54.6)
- added REF**: PinHeader_1x11_P2.54mm_Vertical, Connector_PinHeader_2.54mm:PinHeader_1x11_P2.54mm_Vertical, F.Cu at (207.0, 44.5)
- added REF**: R_Axial_DIN0207_L6.3mm_D2.5mm_P10.16mm_Horizontal, Resistor_THT:R_Axial_DIN0207_L6.3mm_D2.5mm_P10.16mm_Horizontal, F.Cu at (39.4, 64.8)
- added REF**: C_Rect_L7.0mm_W2.0mm_P5.00mm, Capacitor_THT:C_Rect_L7.0mm_W2.0mm_P5.00mm, F.Cu at (52.1, 54.6)
- added REF**: R_Axial_DIN0207_L6.3mm_D2.5mm_P10.16mm_Horizontal, Resistor_THT:R_Axial_DIN0207_L6.3mm_D2.5mm_P10.16mm_Horizontal, F.Cu at (34.3, 57.1)
- added REF**: GPIO 27, Connector_Pin:Pin_D1.0mm_L10.0mm, F.Cu at (227.3, 57.1)
- added REF**: TSOT-23, Package_TO_SOT_SMD:TSOT-23, B.Cu at (43.2, 63.5)
- added REF**: TSOT-23, Package_TO_SOT_SMD:TSOT-23, B.Cu at (43.2, 53.3)
- added REF**: TSOT-23, Package_TO_SOT_SMD:TSOT-23, B.Cu at (43.2, 58.4)
- added REF**: GPIO 26, Connector_Pin:Pin_D1.0mm_L10.0mm, F.Cu at (227.3, 54.6)
- added REF**: Display SCL, Connector_Pin:Pin_D1.0mm_L10.0mm, F.Cu at (257.8, 49.5)
- moved REF** 11.5 mm to (229.9, 31.8)
- moved REF** 3.59 mm to (54.6, 69.9)
- moved DFPLAYER1 2.54 mm to (72.4, 62.2)
- moved REF** 2.54 mm to (52.1, 59.7)
Routing:
- net (no net): track 437.1 -> 459.9 mm, vias 3 -> 36
Other:
- board text added: "1V5 + rt"
- board text added: "25 gn"
- board text added: "25 gn DFPlayer"
- board text added: "26 ge"
- board text added: "26 ge LED"
- board text added: "27 bl"
- board text added: "27 bl Cuckoo"
- board text added: "3V3"
- board text added: "ACHTUNG MOSFET SMD auf Lötseite"
- board text added: "Analoguhr"
- board text added: "BUSY br"
- board text added: "CLK"
- board text added: "CMD"
- board text added: "CN"
- board text added: "Cuckoo bl-sw"
- board text added: "D0"
- board text added: "D1"
- board text added: "D2"
- board text added: "D3"
- board text added: "Display 3V3"
- board text added: "Display SCL"
- board text added: "Display SDA"
- board text added: "GND sw"
- board text added: "GPIO 0"
- board text added: "GPIO 12"
- board text added: "GPIO 13"
- board text added: "GPIO 14"
- board text added: "GPIO 15"
- board text added: "GPIO 16 U2RX"
- board text added: "GPIO 17 U2TX"
- board text added: "GPIO 18"
- board text added: "GPIO 19"
- board text added: "GPIO 2"
- board text added: "GPIO 21"
- board text added: "GPIO 22"
- board text added: "GPIO 23"
- board text added: "GPIO 25"
- board text added: "GPIO 26"
- board text added: "GPIO 27"
- board text added: "GPIO 32"
- board text added: "GPIO 33"
- board text added: "GPIO 34"
- board text added: "GPIO 35"
- board text added: "GPIO 4"
- board text added: "GPIO 5"
- board text added: "LED + ge-rt"
- board text added: "LED ge-sw"
- board text added: "Motor gn-sw"
- board text added: "Q1"
- board text added: "Q2"
- board text added: "Q3"
- board text added: "R1 470"
- board text added: "R10 510"
- board text added: "R11 510"
- board text added: "R12 510"
- board text added: "R13 510"
- board text added: "R2 470"
- board text added: "R3 470"
- board text added: "R4 10k"
- board text added: "R5 10k"
- board text added: "R6 10k"
- board text added: "R7 47"
- board text added: "RESET"
- board text added: "RX ws"
- board text added: "SPK1 + rt"
- board text added: "SPK2 - sw"
- board text added: "TX or"
- board text added: "Touch0"
- board text added: "Touch2"
- board text added: "Touch3"
- board text added: "Touch4"
- board text added: "Treppentaster S2"
- board text added: "VCC 5V0"
- board text added: "VCC rt"
- board text added: "VN"
- board text added: "VP"
- board text added: "Zugschalter S1"
- board text removed: "1,5V Analoguhr"
- board text removed: "5V"
- board text removed: "ACHTUNG MOSFET über Kopf auf Lötseite"
- board text removed: "Cuckoo"
- board text removed: "GPIO 25 26 27"
- board text removed: "LED"
- board text removed: "Motor"
- board text removed: "R1 470 R2 470 R3 470"
- board text removed: "R4 10k R5 10k R6 10k"
- board text removed: "SPK1 +"
- board text removed: "SPK2 -"
- board text removed: "Vin"
- board text removed: "Vout"
